Commit message: Updated project with new features

File: urdf/robot_description.urdf.xacro (robot description, xacro)
@@ -86,9 +86,73 @@
         <origin xyz="0.004419 0.144966 -0.032927" rpy="0 0 0"/>
     </joint>
+    <!--___________________casters___________________-->
+    <link name="caster_front_wheel_link">
+        <inertial>
+            <origin xyz="0.1 0 -0.049389" rpy="0 0 0" />
+            <mass value="1.44379265037902E-06" />
+            <inertia ixx="7.23075276010246E-11" ixy="-6.10956872363424E-16" ixz="2.22849693527207E-15"
+                     iyy="3.87137930859167E-11" iyz="2.939098587861E-15"
+                     izz="1.00967486676306E-10" />
+        </inertial>
+        <origin xyz="0.0 0 0.0" rpy="0 0 0" />
+        <visual>
+            <geometry>
+                <mesh filename="file:///home/kareem/ros2_ws/src/my_robot_description/meshes/f_caster.stl" scale="1.0 1.0 1.0"/>
+            </geometry>
+        </visual>
+        <collision>
+            <origin xyz="0.0 0.0 0.0" rpy="0.0 0.0 0.0"/>
+            <geometry>
+                <mesh filename="file:///home/kareem/ros2_ws/src/my_robot_description/meshes/f_caster.stl" scale="1.0 1.0 1.0"/>
+            </geometry>
+        </collision>
+    </link>
+    <joint name="base_fcaster_wheel_joint" type="fixed">
+        <parent link="base_link" />
+        <child link="caster_front_wheel_link" />
+        <origin xyz="0.1 0 -0.049389" rpy="0 0 0" />
+    </joint>
+    <link name="caster_rear_wheel_link">
+        <origin xyz="0.0 0 0.0" rpy="0 0 0" />
+        <inertial>
+            <origin xyz="-0.121592 0 -0.049389" rpy="0 0 0" />
+            <mass value="1.44379265037902E-06" />
+            <inertia ixx="7.23075276010246E-11" ixy="-6.10956872363424E-16" ixz="2.22849693527207E-15"
+                     iyy="3.87137930859167E-11" iyz="2.939098587861E-15"
+                     izz="1.00967486676306E-10" />
+        </inertial>
+        <visual>
+            <geometry>
+                <mesh filename="file:///home/kareem/ros2_ws/src/my_robot_description/meshes/r_caster.stl" scale="1.0 1.0 1.0"/>
+            </geometry>
+        </visual>
+        <collision>
+            <origin xyz="0.0 0.0 0.0" rpy="0.0 0.0 0.0"/>
+            <geometry>
+                <mesh filename="file:///home/kareem/ros2_ws/src/my_robot_description/meshes/r_caster.stl" scale="1.0 1.0 1.0"/>
+            </geometry>
+        </collision>
+    </link>
+    <joint name="base_rcaster_wheel_joint" type="fixed">
+        <parent link="base_link" />
+        <child link="caster_rear_wheel_link" />
+        <origin xyz="-0.121592 0 -0.049389" rpy="0 0 0" />
+    </joint>
+    <!-- <link name="caster_rear_wheel_link">
+        <origin xyz="-0.1 0 0.016463" rpy="0 0 0" />
+        <visual>
+            <geometry>
+                <sphere radius="0.0164635" />
+            </geometry>
+        </visual>
+    </link>
+    <joint name="base_Rcaster_wheel_joint" type="fixed">
+        <parent link="base_link" />
+        <child link="caster_rear_wheel_link" />
+        <origin xyz="-0.1 0 -0.049389" rpy="0 0 0" />
+    </joint> -->
     <!--______________________________________________________________-->
     <!-- <inertial>
-        <mass value="2.0" />
-        <origin xyz="0 0 0" />
-        <inertia ixx="0.05" ixy="0.0" ixz="0.0" iyy="0.05" iyz="0.0" izz="0.1" />
+       caster wheel 0.032927 dimaeter
     </inertial> -->
 </robot>

File: urdf/robot_description_gazebo.xacro (robot description, xacro)
@@ -19,3 +19,20 @@
         <fdirl>0 1 0</fdirl>
     </gazebo>
+  <!-- Caster Wheels -->
+  <gazebo reference="caster_rear_wheel_link">
+    <mu1>0.1</mu1>
+    <mu2>0.1</mu2>
+    <kp>1000000.0</kp>
+    <kd>100.0</kd>
+    <minDepth>0.001</minDepth>
+    <maxVel>1.0</maxVel>
+  </gazebo>
+  <gazebo reference="caster_front_wheel_link">
+    <mu1>0.1</mu1>
+    <mu2>0.1</mu2>
+    <kp>1000000.0</kp>
+    <kd>100.0</kd>
+    <minDepth>0.001</minDepth>
+    <maxVel>1.0</maxVel>
+  </gazebo>
 </robot>

Commit message: updated with sensors

File: urdf/robot_description.urdf.xacro (robot description, xacro)
@@ -39,5 +39,5 @@
         </inertial>
         <visual>
-            <origin xyz="0.0 0.0 0.0" rpy="0.0 0.0 0.0"/>
+            <origin xyz="0 0 0 " rpy="0.0 0.0 0.0"/>
             <geometry>
                 <mesh filename="file:///home/kareem/ros2_ws/src/my_robot_description/meshes/f_r_wheel.stl" scale="1.0 1.0 1.0"/>
@@ -52,5 +52,5 @@
     </link>
     <!--_________________body & right wheel joint_________________-->
-    <joint name="right_wheel_joint " type="continuous">
+    <joint name="right_wheel_joint" type="continuous">
         <parent link="base_link"/>
         <child link="right_wheel"/>
@@ -66,5 +66,5 @@
         </inertial>
         <visual>
-            <origin xyz="0.0 0.0 0.0" rpy="0.0 0.0 0.0"/>
+            <origin xyz="0 0 0" rpy="0.0 0.0 0.0"/>
             <geometry>
                 <mesh filename="file:///home/kareem/ros2_ws/src/my_robot_description/meshes/f_l_wheel.stl" scale="1.0 1.0 1.0"/>
@@ -80,5 +80,5 @@
     </link>
     <!--___________________body & left wheel joint___________________-->
-    <joint name="left_joint " type="continuous">
+    <joint name="left_wheel_joint" type="continuous">
         <parent link="base_link"/>
         <child link="left_wheel"/>
@@ -139,20 +139,55 @@
         <origin xyz="-0.121592 0 -0.049389" rpy="0 0 0" />
     </joint>
-    <!-- <link name="caster_rear_wheel_link">
-        <origin xyz="-0.1 0 0.016463" rpy="0 0 0" />
+     <!-- __________________________________________________imu link_____________________________________________________________________________-->
+     <link name= "imu_link">
+        <origin xyz="0.0 0 0.12" rpy="0 0 0" />
         <visual>
             <geometry>
-                <sphere radius="0.0164635" />
+                <box size="0.01 0.01 0.01"/>
             </geometry>
+        <collision>
+            <geometry>
+                <box size="0.01 0.01 0.01"/>
+            </geometry>
+        </collision>
+        <inertial>
+            <origin xyz="0.0 0 0.12" rpy="0 0 0" />
+            <mass value="0.001" />
+            <inertia ixx="7.23075276010246E-11" ixy="-6.10956872363424E-16" ixz="2.22849693527207E-15"
+                     iyy="3.87137930859167E-11" iyz="2.939098587861E-15"
+                     izz="1.00967486676306E-10" />
+        </inertial>
         </visual>
     </link>
-    <joint name="base_Rcaster_wheel_joint" type="fixed">
+    <joint name="base_imu_joint" type="fixed">
         <parent link="base_link" />
-        <child link="caster_rear_wheel_link" />
-        <origin xyz="-0.1 0 -0.049389" rpy="0 0 0" />
-    </joint> -->
-    <!--______________________________________________________________-->
-    <!-- <inertial>
-       caster wheel 0.032927 dimaeter
-    </inertial> -->
+        <child link="imu_link" />
+        <origin xyz="0 0 0" rpy="0 0 0" />
+    </joint>
+<!--_______________________________________________________________lidar link________________________________________________________________-->
+    <link name= "lidar">
+        <origin xyz="0.2 0 0.0" rpy="0 0 0" />
+        <visual>
+            <geometry>
+                <cylinder radius="0.001" length="0.001"/>
+            </geometry>
+        <collision>
+            <geometry>
+                <cylinder radius="0.001" length="0.001"/>
+            </geometry>
+        </collision>
+        <inertial>
+            <origin xyz="0.2 0 0.2" rpy="0 0 0" />
+            <mass value="0.001" />
+            <inertia ixx="7.23075276010246E-11" ixy="-6.10956872363424E-16" ixz="2.22849693527207E-15"
+                     iyy="3.87137930859167E-11" iyz="2.939098587861E-15"
+                     izz="1.00967486676306E-10" />
+        </inertial>
+        </visual>
+    </link>
+    <joint name="base_lidar_joint" type="fixed">
+        <parent link="base_link" />
+        <child link="lidar" />
+        <origin xyz="0.15 0 0.0" rpy="0 0 0" />
+    </joint>
 </robot>

File: urdf/robot_description_gazebo.xacro (robot description, xacro)
@@ -36,3 +36,128 @@
     <maxVel>1.0</maxVel>
   </gazebo>
+  <!-- updated-->
+  <!--imu link-->
+  <gazebo reference="imu_link">
+    <sensor name="imu_sensor" type="imu">
+    <plugin filename="libgazebo_ros_imu_sensor.so" name="imu_plugin">
+        <ros>
+          <namespace>/demo</namespace>
+          <remapping>~/out:=imu</remapping>
+        </ros>
+        <initial_orientation_as_reference>false</initial_orientation_as_reference>
+      </plugin>
+      <always_on>true</always_on>
+      <update_rate>100</update_rate>
+      <visualize>true</visualize>
+      <imu>
+        <angular_velocity>
+          <x>
+            <noise type="gaussian">
+              <mean>0.0</mean>
+              <stddev>2e-4</stddev>
+              <bias_mean>0.0000075</bias_mean>
+              <bias_stddev>0.0000008</bias_stddev>
+            </noise>
+          </x>
+          <y>
+            <noise type="gaussian">
+              <mean>0.0</mean>
+              <stddev>2e-4</stddev>
+              <bias_mean>0.0000075</bias_mean>
+              <bias_stddev>0.0000008</bias_stddev>
+            </noise>
+          </y>
+          <z>
+            <noise type="gaussian">
+              <mean>0.0</mean>
+              <stddev>2e-4</stddev>
+              <bias_mean>0.0000075</bias_mean>
+              <bias_stddev>0.0000008</bias_stddev>
+            </noise>
+          </z>
+        </angular_velocity>
+        <linear_acceleration>
+          <x>
+            <noise type="gaussian">
+              <mean>0.0</mean>
+              <stddev>1.7e-2</stddev>
+              <bias_mean>0.1</bias_mean>
+              <bias_stddev>0.001</bias_stddev>
+            </noise>
+          </x>
+          <y>
+            <noise type="gaussian">
+              <mean>0.0</mean>
+              <stddev>1.7e-2</stddev>
+              <bias_mean>0.1</bias_mean>
+              <bias_stddev>0.001</bias_stddev>
+            </noise>
+          </y>
+          <z>
+            <noise type="gaussian">
+              <mean>0.0</mean>
+              <stddev>1.7e-2</stddev>
+              <bias_mean>0.1</bias_mean>
+              <bias_stddev>0.001</bias_stddev>
+            </noise>
+          </z>
+        </linear_acceleration>
+      </imu>
+    </sensor>
+  </gazebo>
+  <!-- diff drive-->
+  <gazebo>
+    <plugin name='diff_drive' filename='libgazebo_ros_diff_drive.so'>
+      <left_joint>left_wheel_joint</left_joint>
+      <right_joint>right_wheel_joint</right_joint>
+      <wheel_separation>0.289932</wheel_separation>
+      <wheel_diameter>0.065</wheel_diameter>
+      <!-- Adjust limits as per your robot's capabilities -->
+      <max_wheel_torque>20</max_wheel_torque> <!-- Maximum torque applied to the wheels -->
+      <max_wheel_accel>1.0</max_wheel_accel> <!-- Maximum acceleration of the wheels -->
+      <!-- Choose whether to publish odometry, odom TF, and wheel TF -->
+      <publish_odom>true</publish_odom> <!-- Whether to publish odometry -->
+      <publish_odom_tf>true</publish_odom_tf> <!-- Whether to publish odometry TF -->
+      <publish_wheel_tf>true</publish_wheel_tf> <!-- Whether to publish wheel TF -->
+      <!-- Update frame names according to your robot's URDF -->
+      <odometry_frame>odom</odometry_frame> <!-- Frame for odometry data -->
+      <robot_base_frame>base_footprint</robot_base_frame> <!-- Base frame of the robot -->
+    </plugin>
+  </gazebo>
+  <!-- lidar -->
+  <gazebo reference="lidar">
+    <sensor name="gazebo_lidar" type="ray">
+      <pose>0 0 0 0 0 0</pose>
+      <always_on>true</always_on>
+      <visualize>true</visualize>
+      <update_rate>10.0</update_rate>
+      <plugin filename="libgazebo_ros_ray_sensor.so" name="gazebo_lidar">
+          <ros>
+            <remapping>~/out:=scan</remapping>
+          </ros>
+          <output_type>sensor_msgs/LaserScan</output_type>
+          <frame_name>lidar</frame_name>
+      </plugin>
+      <ray>
+        <scan>
+          <horizontal>
+            <samples>360</samples>
+            <resolution>1</resolution>
+            <min_angle>-3.14</min_angle>
+            <max_angle>3.14</max_angle>
+          </horizontal>
+        </scan>
+        <range>
+          <min>0.120</min>
+          <max>3.5</max>
+          <resolution>0.015</resolution>
+        </range>
+        <noise>
+          <type>gaussian</type>
+          <mean>0.0</mean>
+          <stddev>0.01</stddev>
+        </noise>
+      </ray>
+    </sensor>
+  </gazebo>
 </robot>

Commit message: t

File: urdf/robot_description.urdf.xacro (robot description, xacro)
@@ -15,5 +15,5 @@
             <origin xyz="0.0 0.0 0.0" rpy="0.0 0.0 0.0"/>
             <geometry>
-                <mesh filename="file:///home/kareem/ros2_ws/src/my_robot_description/meshes/f_body.stl" scale="1.0 1.0 1.0"/>
+                <mesh filename="$(find my_robot_description)/meshes/f_body.stl" scale="1.0 1.0 1.0"/>
             </geometry>
         </visual>
@@ -21,5 +21,5 @@
             <origin xyz="0.0 0.0 0.0" rpy="0.0 0.0 0.0"/>
             <geometry>
-                <mesh filename="file:///home/kareem/ros2_ws/src/my_robot_description/meshes/f_body.stl" scale="1.0 1.0 1.0"/>
+                <mesh filename="$(find my_robot_description)/meshes/f_body.stl" scale="1.0 1.0 1.0"/>
             </geometry>
         </collision>
@@ -41,5 +41,5 @@
             <origin xyz="0 0 0 " rpy="0.0 0.0 0.0"/>
             <geometry>
-                <mesh filename="file:///home/kareem/ros2_ws/src/my_robot_description/meshes/f_r_wheel.stl" scale="1.0 1.0 1.0"/>
+                <mesh filename="$(find my_robot_description)/meshes/f_r_wheel.stl" scale="1.0 1.0 1.0"/>
             </geometry>
         </visual>
@@ -47,5 +47,5 @@
             <origin xyz="0.0 0.0 0.0" rpy="0.0 0.0 0.0"/>
             <geometry>
-                <mesh filename="file:///home/kareem/ros2_ws/src/my_robot_description/meshes/f_r_wheel.stl" scale="1.0 1.0 1.0"/>
+                <mesh filename="$(find my_robot_description)/meshes/f_r_wheel.stl" scale="1.0 1.0 1.0"/>
             </geometry>
         </collision>
@@ -68,5 +68,5 @@
             <origin xyz="0 0 0" rpy="0.0 0.0 0.0"/>
             <geometry>
-                <mesh filename="file:///home/kareem/ros2_ws/src/my_robot_description/meshes/f_l_wheel.stl" scale="1.0 1.0 1.0"/>
+                <mesh filename="$(find my_robot_description)/meshes/f_l_wheel.stl" scale="1.0 1.0 1.0"/>
             </geometry>
         </visual>
@@ -75,5 +75,5 @@
             <origin xyz="0.0 0.0 0.0" rpy="0.0 0.0 0.0"/>
             <geometry>
-                <mesh filename="file:///home/kareem/ros2_ws/src/my_robot_description/meshes/f_l_wheel.stl" scale="1.0 1.0 1.0"/>
+                <mesh filename="$(find my_robot_description)/meshes/f_l_wheel.stl" scale="1.0 1.0 1.0"/>
             </geometry>
         </collision>
@@ -98,5 +98,5 @@
         <visual>
             <geometry>
-                <mesh filename="file:///home/kareem/ros2_ws/src/my_robot_description/meshes/f_caster.stl" scale="1.0 1.0 1.0"/>
+                <mesh filename="$(find my_robot_description)/meshes/f_caster.stl" scale="1.0 1.0 1.0"/>
             </geometry>
         </visual>
@@ -104,5 +104,5 @@
             <origin xyz="0.0 0.0 0.0" rpy="0.0 0.0 0.0"/>
             <geometry>
-                <mesh filename="file:///home/kareem/ros2_ws/src/my_robot_description/meshes/f_caster.stl" scale="1.0 1.0 1.0"/>
+                <mesh filename="$(find my_robot_description)/meshes/f_caster.stl" scale="1.0 1.0 1.0"/>
             </geometry>
         </collision>
@@ -124,5 +124,5 @@
         <visual>
             <geometry>
-                <mesh filename="file:///home/kareem/ros2_ws/src/my_robot_description/meshes/r_caster.stl" scale="1.0 1.0 1.0"/>
+                <mesh filename="$(find my_robot_description)/meshes/r_caster.stl" scale="1.0 1.0 1.0"/>
             </geometry>
         </visual>
@@ -130,5 +130,5 @@
             <origin xyz="0.0 0.0 0.0" rpy="0.0 0.0 0.0"/>
             <geometry>
-                <mesh filename="file:///home/kareem/ros2_ws/src/my_robot_description/meshes/r_caster.stl" scale="1.0 1.0 1.0"/>
+                <mesh filename="$(find my_robot_description)/meshes/r_caster.stl" scale="1.0 1.0 1.0"/>
             </geometry>
         </collision>
